File: tests/board_samples/kicad_6/missing.kicad_sch (KiCad schematic)
At the start: 4 parts

Commit message: Adjusted error messages and crossed comp generation.
- Also the name of the member for lib_name
Parts:
- R1: symbol Resistor -> A:B:Resistor
Changed lines of the file:
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@@
     )
   )
-  (symbol (lib_id "Resistor") (at 53.34 43.18 0) (unit 1)
+  (symbol (lib_id "A:B:Resistor") (at 53.34 43.18 0) (unit 1)
     (in_bom yes) (on_board yes)
     (property "Reference" "R1" (id 0) (at 55.118 42.0116 0)
