File: tests/board_samples/kicad_6/links.kicad_sch (KiCad schematic)
At the start: 4 parts, among them J1 Molex KK ñoño, J2 Molex KK

Commit message: [BoM][Added] Option to link to Mouser site.
Parts:
- C1: mouser# (none) -> 80-C0805C102K5R; mouser_alt# (none) -> 80-C0805C102K5R7210
- J1, J2: mouser# (none) -> 538-22-23-2021; mouser_alt# (none) -> 538-22-11-2022
- R1: mouser# (none) -> 652-CR0805JW-102ELF; mouser_alt# (none) -> 652-CRS0805JX102ELF
Changed lines of the file:
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@@
+      (effects (font (size 1.27 1.27)) hide)
+    )
+    (property "mouser#" "538-22-23-2021" (id 4) (at 72.39 58.42 0)
+      (effects (font (size 1.27 1.27)) hide)
+    )
+    (property "mouser_alt#" "538-22-11-2022" (id 4) (at 72.39 58.42 0)
       (effects (font (size 1.27 1.27)) hide)
     )
@@
       (effects (font (size 1.27 1.27)) hide)
     )
+    (property "mouser#" "538-22-23-2021" (id 4) (at 72.39 58.42 0)
+      (effects (font (size 1.27 1.27)) hide)
+    )
+    (property "mouser_alt#" "538-22-11-2022" (id 4) (at 72.39 58.42 0)
+      (effects (font (size 1.27 1.27)) hide)
+    )
     (pin "1")
     (pin "2")
@@
     )
     (property "digikey_alt#" "CRS0805-JX-102ELFCT-ND" (id 6) (at 87.63 58.42 90)
+      (effects (font (size 1.27 1.27)) hide)
+    )
+    (property "mouser#" "652-CR0805JW-102ELF" (id 4) (at 72.39 58.42 0)
+      (effects (font (size 1.27 1.27)) hide)
+    )
+    (property "mouser_alt#" "652-CRS0805JX102ELF" (id 4) (at 72.39 58.42 0)
       (effects (font (size 1.27 1.27)) hide)
     )
@@
       (effects (font (size 1.27 1.27)) hide)
     )
+    (property "mouser#" "80-C0805C102K5R" (id 4) (at 72.39 58.42 0)
+      (effects (font (size 1.27 1.27)) hide)
+    )
+    (property "mouser_alt#" "80-C0805C102K5R7210" (id 4) (at 72.39 58.42 0)
+      (effects (font (size 1.27 1.27)) hide)
+    )

Commit message: [BoM][Added] LCSC links
From SchrodingersGat/KiBoM#190
Parts:
- C1: LCSC# (none) -> C2167366
- J1, J2: LCSC# (none) -> C234180
- R1: LCSC# (none) -> C840623
Changed lines of the file:
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@@
+      (effects (font (size 1.27 1.27)) hide)
+    )
+    (property "LCSC#" "C234180" (at 72.39 58.42 0)
       (effects (font (size 1.27 1.27)) hide)
     )
@@
       (effects (font (size 1.27 1.27)) hide)
     )
+    (property "LCSC#" "C234180" (at 72.39 58.42 0)
+      (effects (font (size 1.27 1.27)) hide)
+    )
     (pin "1")
     (pin "2")
@@
     )
     (property "mouser_alt#" "652-CRS0805JX102ELF" (id 4) (at 72.39 58.42 0)
+      (effects (font (size 1.27 1.27)) hide)
+    )
+    (property "LCSC#" "C840623" (at 72.39 58.42 0)
       (effects (font (size 1.27 1.27)) hide)
     )
@@
       (effects (font (size 1.27 1.27)) hide)
     )
+    (property "LCSC#" "C2167366" (at 72.39 58.42 0)
+      (effects (font (size 1.27 1.27)) hide)
+    )
