File: tests/board_samples/kicad_6/batteryPack.kicad_pcb (KiCad board)
At the start: 2 copper layers, 204 x 78 mm, 48 parts, among them J1 Mirco USB, J10 B1+, J11 B1-, J12 B2-, J13 B1+, J14 B1-, J15 B2+, J16 B2-, J2 B1+, J3 B1-, J4 B2-, J5 B2+, J6 CableConnector, J7 SWD, J8 UART, J9 B2+, P1 USB-C, U1 TP5100-Module, U2 STM32F030F4Px, U3 XC6206P332MR, U4 TP5100-Module

Commit message: [Tests][PCB2Blender][Added] Stacked boards and JSON stack-up
Other:
- board text added: "PCB3D_BR_BConn"
- board text added: "PCB3D_BR_BPack"
- board text added: "PCB3D_BR_Charger"
- board text added: "PCB3D_STACK_BConn_ONTO_BPack_25"
- board text added: "PCB3D_TL_BConn"
- board text added: "PCB3D_TL_BPack"
- board text added: "PCB3D_TL_Charger"
Changed lines of the file:
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@@
     (effects (font (size 5 5) (thickness 0.5)))
+  )
+  (gr_text "PCB3D_BR_BConn" (at 137.25 90.75) (layer "Eco2.User")
+    (effects (font (size 1.5 1.5) (thickness 0.3) bold) (justify left bottom))
+  )
+  (gr_text "PCB3D_BR_BPack" (at 70.25 109.75) (layer "Eco2.User")
+    (effects (font (size 1.5 1.5) (thickness 0.3) bold) (justify left bottom))
+  )
+  (gr_text "PCB3D_STACK_BConn_ONTO_BPack_25" (at 36.25 53.75) (layer "Eco2.User")
+    (effects (font (size 1.5 1.5) (thickness 0.3) bold) (justify left bottom))
+  )
+  (gr_text "PCB3D_TL_BConn" (at 116.25 47.75) (layer "Eco2.User")
+    (effects (font (size 1.5 1.5) (thickness 0.3) bold) (justify left bottom))
+  )
+  (gr_text "PCB3D_TL_BPack" (at 29.25 29.75) (layer "Eco2.User")
+    (effects (font (size 1.5 1.5) (thickness 0.3) bold) (justify left bottom))
+  )
+  (gr_text "PCB3D_BR_Charger" (at 235.25 89.75) (layer "Eco2.User")
+    (effects (font (size 1.5 1.5) (thickness 0.3) bold) (justify left bottom))
+  )
+  (gr_text "PCB3D_TL_Charger" (at 186.25 50.75) (layer "Eco2.User")
+    (effects (font (size 1.5 1.5) (thickness 0.3) bold) (justify left bottom))
   )
   (dimension (type aligned) (layer "F.Fab")
