File: tests/board_samples/kicad_7/test_v5.kicad_sch (KiCad schematic)
At the start: 4 parts

Commit message: [Tests] Adapted to the new behavior
- Removed bogus componentes in test_v5 PCBs
- Accounted for R3 in kibom-variant_3 PCB
Parts:
- C1, L1: footprint (none) -> Capacitor_SMD:C_0805_2012Metric
- R1, R2: footprint (none) -> Resistor_SMD:R_0805_2012Metric
Changed lines of the file:
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@@
       (effects (font (size 1.27 1.27)))
     )
-    (property "Footprint" "" (at 33.02 85.852 90)
+    (property "Footprint" "Resistor_SMD:R_0805_2012Metric" (at 33.02 85.852 90)
       (effects (font (size 1.27 1.27)) hide)
     )
@@
       (effects (font (size 1.27 1.27)) (justify left))
     )
-    (property "Footprint" "" (at 39.37 80.01 0)
+    (property "Footprint" "Capacitor_SMD:C_0805_2012Metric" (at 39.37 80.01 0)
       (effects (font (size 1.27 1.27)) hide)
     )
@@
       (effects (font (size 1.27 1.27)))
     )
-    (property "Footprint" "" (at 49.53 86.6648 0)
+    (property "Footprint" "Capacitor_SMD:C_0805_2012Metric" (at 49.53 86.6648 0)
       (effects (font (size 1.27 1.27)) hide)
     )
@@
       (effects (font (size 1.27 1.27)) (justify right))
     )
-    (property "Footprint" "" (at 38.354 94.996 90)
+    (property "Footprint" "Resistor_SMD:R_0805_2012Metric" (at 38.354 94.996 90)
       (effects (font (size 1.27 1.27)) hide)
     )
