File: tests/board_samples/kicad_8/rotations.kicad_sch (KiCad schematic)
At the start: 8 parts, among them Q1 Q_NPN_BCE, Q2 Q_NPN_BCE, Q3 Q_NPN_BCE, Q4 Q_NPN_BCE, Q5 Q_NPN_BCE, Q6 Q_NPN_BCE, Q7 Q_NPN_BCE, Q8 Q_NPN_BCE

Commit message: [Globals][Added] use_pcb_fields
Allows using fields defined in the PCB (and not only in the schematic),
enabled by default

See #648 and #650
Parts:
- Q3: JLCRotOffset 270 -> (none)
Other:
- note added: "Q3 is rotated using a field only found in the PCB"
Changed lines of the file:
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@@
 	(generator_version "8.0")
 	(paper "A4")
+	(text "Q3 is rotated using a field\nonly found in the PCB"
+		(exclude_from_sim no)
+		(at 110.49 40.894 0)
+		(effects
+			(font
+				(size 1.27 1.27)
+			)
+		)
+	)
 	(symbol
 		(lib_id "Device:Q_NPN_BCE")
@@
 			(at 106.68 50.8 0)
 			(effects
-				(font
-					(size 1.27 1.27)
-				)
-				(hide yes)
-			)
-		)
-		(property "JLCRotOffset" "270"
-			(at 106.68 50.8 0)
-			(effects
